Commit message: Correct weight

File: rossumo_description/urdf/rossumo.xacro (robot description, xacro)
@@ -16,10 +16,10 @@
     <pose>0 0 0.1 0 0 0</pose>
     <inertial>
-      <mass value="0.14"/>
+      <mass value="0.16"/>
         <origin xyz="0.0 0 0.055" rpy="0 0 0"/>
       <inertia
-          ixx="0.0004" ixy="0.00" ixz="0.00"
-          iyy="0.0004" iyz="0.00"
-          izz="0.0004"
+          ixx="0.00036" ixy="0.00" ixz="0.00"
+          iyy="0.00036" iyz="0.00"
+          izz="0.00036"
       />
     </inertial>
